File: Schematics/Ballmouse.kicad_pcb (KiCad board)
At the start: 2 copper layers, 49.2 x 71.6 mm, 38 parts, among them J1 Conn_01x06, J11 USB_C_Plug_USB2.0, J2 Conn_01x06, Q1 PMOS, SW1 SW_SPST, SW2 SW_SPST, SW3 SW_SPST, SW4 SW_SPST, SW5 SW_SPST, U1 PMW3360DM-T2QU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

Commit message: Ready to order PCB
Parts:
- added D3: WS2812B, UE_LED:SK6812-E_FaceUp, F.Cu at (139.2, 82.8)
- added D4: WS2812B, UE_LED:SK6812-E_FaceUp, F.Cu at (127.6, 95.6)
- added D5: WS2812B, UE_LED:SK6812-E_FaceUp, F.Cu at (139.2, 108.1)
- added D6: WS2812B, UE_LED:SK6812-E_FaceUp, F.Cu at (151.0, 95.6)
- moved kibuzzard-691E3A0F 13.2 mm to (132.0, 122.4)
- moved C12 3.40 mm to (151.8, 91.6)
- moved C11 3.20 mm to (151.7, 89.2)
Connections:
- U2 pad 3: unconnected-(U2-PC14-Pad3) -> Neo
Routing:
- net +5V: track 70.8 -> 142.9 mm
- net Net-(D5-DOUT): track 0.00 -> 23.4 mm
- net Net-(D4-DOUT): track 0.00 -> 18.7 mm
- net Net-(D3-DOUT): track 0.00 -> 16.2 mm, vias 0 -> 2
- net Neo: track 0.00 -> 9.76 mm, vias 0 -> 2
- net +1V8: track 34.6 -> 30.0 mm
