File: Schematics/Ballmouse.kicad_sch (KiCad schematic)
At the start: 21 parts, among them J11 USB_C_Plug_USB2.0, Q1 PMOS, U1 PMW3360DM-T2QU, U2 STM32F072C8Tx, U3 TLV1117-33, U4 XC6206-1.8NR

Commit message: Unrouted:0. Should I add leds?
Parts:
- added D1, D2: LED_Small, LED_SMD:LED_0805_2012Metric, symbol Device:LED_Small
- added H1, H2, H3, H4: MountingHole, UE_Standoff:M3ThreadedStandoff, symbol Mechanical:MountingHole
- added J1: Conn_01x06, Connector_PinHeader_1.27mm:PinHeader_1x06_P1.27mm_Vertical, symbol Connector_Generic:Conn_01x06
- added J2: Conn_01x06, Connector_PinHeader_2.54mm:PinHeader_1x06_P2.54mm_Vertical, symbol Connector_Generic:Conn_01x06
- added RN2: 330, Resistor_SMD:R_Array_Convex_4x0603, symbol Device:R_Pack04
- added SW1, SW2, SW3, SW4, SW5: SW_SPST, UE_Buttons:TS3315A, symbol Switch:SW_SPST
- C1, C11, C12, C2, C3, C4, C5: footprint (none) -> Capacitor_SMD:C_0805_2012Metric
- C16, C8: footprint Capacitor_SMD:C_0805_2012Metric -> Capacitor_SMD:C_0603_1608Metric
- R1: footprint (none) -> Resistor_SMD:R_0805_2012Metric
- U1: footprint (none) -> UE_Module:PMW3360
- U4: footprint Package_TO_SOT_SMD:SOT-223-3_TabPin2 -> Package_TO_SOT_SMD:SOT-23
Connections:
- net D+: now also U2.33 (PA12)
- net D-: now also U2.32 (PA11)
- net Led_power: now also U2.2 (PC13)
- net MISO: now also U2.16 (PA6)
- net MOSI: now also U2.17 (PA7)
- net Motion: now also U2.12 (PA2)
- net SCLK: now also U2.15 (PA5)
- net VCC: now also U2.1 (VBAT), J2.1 (Pin_1)
- net VSS: now also D1.1 (K), D2.1 (K), J2.4 (Pin_4), SW1.2 (B), SW2.2 (B), SW3.2 (B), SW4.2 (B), SW5.2 (B)
- net ~{CS}: now also U2.14 (PA4)
- net 3360_Reset: now reaches U1.7 (~{RESET})
- net 3360_Reset: now also U2.11 (PA1)
- net at RN1.7 (R2.2): now also J11.B5 (CC2); no longer J11.A5 (CC1)
- net at RN1.8 (R1.2): now also J11.A5 (CC1); no longer J11.B5 (CC2)
- net Five: now reaches U2.13 (PA3)
- net Five: now also SW5.1 (A)
- net at U2.18 (PB0): now also RN2.2 (R2.1)
- net at U2.19 (PB1): now also RN2.1 (R1.1)
- net at U2.21 (PB10): now also J1.1 (Pin_1)
- net at U2.22 (PB11): now also J1.2 (Pin_2)
- net at U2.25 (PB12): now also J1.3 (Pin_3)
- net at U2.26 (PB13): now also J1.4 (Pin_4)
- net at U2.27 (PB14): now also J1.5 (Pin_5)
- net at U2.28 (PB15): now also J1.6 (Pin_6)
- net SWDIO: now reaches U2.34 (PA13)
- net SWDIO: now also J2.6 (Pin_6)
- net SWCLK: now reaches U2.37 (PA14)
- net SWCLK: now also J2.5 (Pin_5)
- net One: now reaches U2.40 (PB4)
- net One: now also SW1.1 (A)
- net Two: now reaches U2.41 (PB5)
- net Two: now also SW2.1 (A)
- net Three: now reaches U2.42 (PB6)
- net Three: now also SW3.1 (A)
- net Four: now reaches U2.43 (PB7)
- net Four: now also SW4.1 (A)
- net Boot: now reaches U2.44 (BOOT0)
- net Boot: now also J2.3 (Pin_3)
- net Reset: now reaches U2.7 (NRST)
- net Reset: now also J2.2 (Pin_2)
- new net: D1.2 (A), RN2.7 (R2.2)
- new net: D2.2 (A), RN2.8 (R1.2)
- no-connect marks 6 -> 10
Other:
- moved on the sheet: C1, C10, C16, C2, C3, C4, C5, C6, C7, C8, C9, RN1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

Commit message: Ready to order PCB
Parts:
- added D3, D4, D5, D6: WS2812B, UE_LED:SK6812-E_FaceUp, symbol LED:WS2812B
Connections:
- net +5V: now also D3.1 (VDD), D4.1 (VDD), D5.1 (VDD), D6.1 (VDD)
- net VSS: now also D3.3 (VSS), D4.3 (VSS), D5.3 (VSS), D6.3 (VSS)
- net Neo: now reaches U2.3 (PC14)
- net Neo: now also D3.4 (DIN)
- new net: D5.2 (DOUT), D6.4 (DIN)
- new net: D4.2 (DOUT), D5.4 (DIN)
- new net: D3.2 (DOUT), D4.4 (DIN)
Other:
- moved on the sheet: C11, C12, Q1, R1, U1
